Commit message: update

File: assets/mounted_bh_282.urdf (robot description, URDF)
Before this commit: robot , 21 links, 20 joints
Joints:
- joint bh_j11_joint: origin xyz=-0.02500 0.00000 0.02520 rpy=0.00000 -0.00000 1.57080 -> xyz=-0.02500 0.00000 0.02520 rpy=0.00000 0.00000 1.57080
- joint bh_j21_joint: origin xyz=0.02500 0.00000 0.02520 rpy=0.00000 -0.00000 1.57080 -> xyz=0.02500 0.00000 0.02520 rpy=0.00000 0.00000 1.57080

Commit message: update

File: assets/mounted_bh_282.urdf (robot description, URDF)
Before this commit: robot , 21 links, 20 joints
Joints:
- joint bh_j11_joint: origin xyz=-0.02500 0.00000 0.02520 rpy=0.00000 0.00000 1.57080 -> xyz=-0.02500 0.00000 0.02520 rpy=0.00000 -0.00000 1.57080
- joint bh_j21_joint: origin xyz=0.02500 0.00000 0.02520 rpy=0.00000 0.00000 1.57080 -> xyz=0.02500 0.00000 0.02520 rpy=0.00000 -0.00000 1.57080
