Commit message: updated robot files

File: dofbot_pro_ws/src/dofbot_pro_v24/urdf/DOFBOT_Pro-V24.urdf (robot description, URDF)
Before this commit: robot DOFBOT_Pro-V24, 14 links, 13 joints
Links:
- link Arm1_Link: geometry collision mesh filename=package://dofbot_pro_v24/meshes/Arm1_Link.STL; visual mesh filename=package://dofbot_pro_v24/meshes/Arm1_Link.STL
- link Arm2_Link: geometry collision mesh filename=package://dofbot_pro_v24/meshes/Arm2_Link.STL; visual mesh filename=package://dofbot_pro_v24/meshes/Arm2_Link.STL
- link Arm3_Link: geometry collision mesh filename=package://dofbot_pro_v24/meshes/Arm3_Link.STL; visual mesh filename=package://dofbot_pro_v24/meshes/Arm3_Link.STL
- link Arm4_Link: geometry collision mesh filename=package://dofbot_pro_v24/meshes/Arm4_Link.STL; visual mesh filename=package://dofbot_pro_v24/meshes/Arm4_Link.STL
- link Arm5_Link: geometry collision mesh filename=package://dofbot_pro_v24/meshes/Arm5_Link.STL; visual mesh filename=package://dofbot_pro_v24/meshes/Arm5_Link.STL
- link DaBai_DCW2_Link: geometry collision mesh filename=package://dofbot_pro_v24/meshes/DaBai_DCW2_Link.STL; visual mesh filename=package://dofbot_pro_v24/meshes/DaBai_DCW2_Link.STL
- link Gripping_point_Link: geometry collision mesh filename=package://dofbot_pro_v24/meshes/Gripping_point_Link.STL; visual mesh filename=package://dofbot_pro_v24/meshes/Gripping_point_Link.STL
- link base_link: geometry collision mesh filename=package://dofbot_pro_v24/meshes/base_link.STL; visual mesh filename=package://dofbot_pro_v24/meshes/base_link.STL
- link llink1: geometry collision mesh filename=package://dofbot_pro_v24/meshes/llink1.STL; visual mesh filename=package://dofbot_pro_v24/meshes/llink1.STL
- link llink2: geometry collision mesh filename=package://dofbot_pro_v24/meshes/llink2.STL; visual mesh filename=package://dofbot_pro_v24/meshes/llink2.STL
- link llink3: geometry collision mesh filename=package://dofbot_pro_v24/meshes/llink3.STL; visual mesh filename=package://dofbot_pro_v24/meshes/llink3.STL
- link rlink1: geometry collision mesh filename=package://dofbot_pro_v24/meshes/rlink1.STL; visual mesh filename=package://dofbot_pro_v24/meshes/rlink1.STL
- link rlink2: geometry collision mesh filename=package://dofbot_pro_v24/meshes/rlink2.STL; visual mesh filename=package://dofbot_pro_v24/meshes/rlink2.STL
- link rlink3: geometry collision mesh filename=package://dofbot_pro_v24/meshes/rlink3.STL; visual mesh filename=package://dofbot_pro_v24/meshes/rlink3.STL
